Commit message: fix model and launch (added dummy gripper and dummy base)

File: rm_63_b_description/urdf/rm_63_b_base_description.urdf (robot description, URDF)
Before this commit: robot rm_63_b_description, 12 links, 11 joints
Links:
- link base_footprint: geometry collision cylinder length=0.2 radius=0.25; visual cylinder length=0.2 radius=0.25
Joints:
- joint fixed_joint_base: origin xyz=0 0 0 rpy=0 0 0 -> xyz=0 0 0.2 rpy=0 0 0
