Commit message: change dummy base to fit turtlebot3 waffle

File: rm_63_b_description/urdf/rm_63_b_dummy_base_description.urdf (robot description, URDF)
Before this commit: robot rm_63_b_description, 12 links, 11 joints
Links:
- link base_footprint: geometry collision box size=0.3 0.26 0.142; visual box size=0.3 0.26 0.142
Joints:
- joint fixed_joint_base: origin xyz=0 0 0.2 rpy=0 0 0 -> xyz=0 0 0.1425 rpy=0 0 0
