Commit message: ADD moveit_config pkg

File: rm_63_b_description/urdf/rm_63_b.urdf (robot description, URDF)
Before this commit: robot rm_63_b_description, 12 links, 11 joints
Links:
- link base_footprint: geometry 
Joints:
- joint fixed_joint_base: origin xyz=0 0 0.1425 rpy=0 0 0 -> xyz=0 0 0 rpy=0 0 0

File: rm_63_b_description/urdf/rm_63_b_dummy_base.urdf (robot description, URDF)
Before this commit: robot rm_63_b_description, 12 links, 11 joints
Links:
- link base_footprint: geometry collision box size=0.3 0.26 0.142; visual box size=0.3 0.26 0.142
Joints:
- joint fixed_joint_base: origin xyz=0 0 0 rpy=0 0 0 -> xyz=0 0 0.1425 rpy=0 0 0

Commit message: fix gripper

File: rm_63_b_description/urdf/rm_63_b.urdf (robot description, URDF)
Before this commit: robot rm_63_b, 12 links, 11 joints
Links:
- link gripper_base: geometry collision cylinder length=0.04 radius=0.02; visual cylinder length=0.04 radius=0.02
- link gripper_left_finger: geometry collision box size=0.01 0.04 0.1; visual box size=0.01 0.04 0.1
- link gripper_palm: geometry collision box size=0.11 0.06 0.02; visual box size=0.11 0.06 0.02
- link gripper_right_finger: geometry collision box size=0.01 0.04 0.1; visual box size=0.01 0.04 0.1
Joints:
- joint base_to_palm: origin xyz=0 0 0.03 -> xyz=0.04 0 0 rpy=1.57080 0 1.57080
- joint joint6: limit lower=-6.28 upper=6.28 effort=100 velocity=1 -> lower=-3.106 upper=3.106 effort=100 velocity=1
- joint manipulator_to_gripper: origin xyz=0 0 0 -> xyz=0 0 0 rpy=0 -1.57080 0
- joint palm_to_left_finger: limit lower=0 upper=0.03 effort=1.0 velocity=0.5 -> lower=0 upper=0.045 effort=1.0 velocity=0.5
- joint palm_to_right_finger: limit lower=0 upper=0.03 effort=1.0 velocity=0.5 -> lower=0 upper=0.045 effort=1.0 velocity=0.5

File: rm_63_b_description/urdf/rm_63_b_dummy_base.urdf (robot description, URDF)
Before this commit: robot rm_63_b_dummy_base, 12 links, 11 joints
Links:
- link gripper_base: geometry collision cylinder length=0.04 radius=0.02; visual cylinder length=0.04 radius=0.02
- link gripper_left_finger: geometry collision box size=0.01 0.04 0.1; visual box size=0.01 0.04 0.1
- link gripper_palm: geometry collision box size=0.11 0.06 0.02; visual box size=0.11 0.06 0.02
- link gripper_right_finger: geometry collision box size=0.01 0.04 0.1; visual box size=0.01 0.04 0.1
Joints:
- joint base_to_palm: origin xyz=0 0 0.03 -> xyz=0.04 0 0 rpy=1.57080 0 1.57080
- joint joint6: limit lower=-6.28 upper=6.28 effort=100 velocity=1 -> lower=-3.106 upper=3.106 effort=100 velocity=1
- joint manipulator_to_gripper: origin xyz=0 0 0 -> xyz=0 0 0 rpy=0 -1.57080 0
- joint palm_to_left_finger: limit lower=0 upper=0.03 effort=1.0 velocity=0.5 -> lower=0 upper=0.045 effort=1.0 velocity=0.5
- joint palm_to_right_finger: limit lower=0 upper=0.03 effort=1.0 velocity=0.5 -> lower=0 upper=0.045 effort=1.0 velocity=0.5
